Commit message: simulation 11.22

File: clober_ros2/clober_description/urdf/clober_gazebo.urdf.xacro (robot description, xacro)
@@ -26,4 +26,11 @@
     <color rgba="0.15 0.15 0.15 1.0" />
   </material>
+<!--
+  <link name="map">
+  <joint name="base_joint" type="fixed">
+    <parent link="map" />
+    <child link="base_link" />
+    <origin xyz="0 0 0" rpy="0 0 0" />
+  </joint> -->
   <link name="base_link">
     <visual>

Commit message: change laser_tf for multimap

File: clober_ros2/clober_description/urdf/clober_gazebo.urdf.xacro (robot description, xacro)
@@ -27,7 +27,7 @@
   </material>
 <!--
-  <link name="map">
+  <link name="base_footprint">
   <joint name="base_joint" type="fixed">
-    <parent link="map" />
+    <parent link="base_footprint" />
     <child link="base_link" />
     <origin xyz="0 0 0" rpy="0 0 0" />
